File: 36k.kicad_pcb (KiCad board)
At the start: 2 copper layers, 115.7 x 95.8 mm, 84 parts, among them J1 MJ-4PP-9, J2 OLED, J3 MJ-4PP-9, J4 OLED, SW1 SW_PUSH, SW10 SW_PUSH, SW11 SW_PUSH, SW12 SW_PUSH, SW13 SW_PUSH, SW14 SW_PUSH, SW15 SW_PUSH, SW16 SW_PUSH, SW17 SW_PUSH, SW18 SW_PUSH, SW19 SW_PUSH, SW2 SW_PUSH, SW20 SW_PUSH, SW21 SW_PUSH, SW22 SW_PUSH, SW23 SW_PUSH, SW24 SW_PUSH, SW25 SW_PUSH, SW26 SW_PUSH, SW27 SW_PUSH, SW28 SW_PUSH, SW29 SW_PUSH, SW3 SW_PUSH, SW30 SW_PUSH, SW31 SW_PUSH, SW32 SW_PUSH, SW33 SW_PUSH, SW34 SW_PUSH, SW35 SW_PUSH, SW36 SW_PUSH, SW4 SW_PUSH, SW5 SW_PUSH, SW6 SW_PUSH, SW7 SW_PUSH, SW8 SW_PUSH, SW9 SW_PUSH, U1 ProMicro, U2 ProMicro

Commit message: changes
Parts:
- BT1, BT2: moved to B.Cu
- RSW2: footprint kbd:Power -> Button_Switch_THT:SW_CuK_OS102011MA1QN1_SPDT_Angled
- RSW4: footprint kbd:Power -> Button_Switch_THT:SW_CuK_OS102011MA1QN1_SPDT_Angled; moved to B.Cu
- moved RSW2 72.4 mm to (132.1, 137.2)
- moved J3 30.1 mm to (134.6, 109.5)
- moved U2 27.9 mm to (143.6, 82.0)
- moved J4 27.3 mm to (139.8, 102.6)
- moved RSW3 26.3 mm to (136.3, 101.5), turned to 90 degrees
- moved BT2 23.5 mm to (151.7, 103.2)
- moved RSW4 10.5 mm to (162.6, 99.1)
- moved J1 4.37 mm to (130.3, 109.4)
- moved BT1 4.23 mm to (113.1, 103.1), turned to 0 degrees
- moved RSW1 2.83 mm to (128.6, 101.5)
Routing:
- net raw: track 0.00 -> 40.2 mm, vias 0 -> 1
- net GND: track 52.6 -> 43.6 mm
- net data: track 0.00 -> 4.40 mm, vias 0 -> 1
- net VCC: track 49.4 -> 45.0 mm
- net row2: track 119.3 -> 121.2 mm
- net row3: track 81.7 -> 83.3 mm
- net reset: track 41.7 -> 43.2 mm, vias 2 -> 1
Other:
- board size 115.7 x 95.8 mm -> 234.5 x 95.8 mm
