File: 36k.kicad_sch (KiCad schematic)
At the start: 84 parts, among them J1 MJ-4PP-9, J2 OLED, J3 MJ-4PP-9, J4 OLED, SW1 SW_PUSH, SW10 SW_PUSH, SW11 SW_PUSH, SW12 SW_PUSH, SW13 SW_PUSH, SW14 SW_PUSH, SW15 SW_PUSH, SW16 SW_PUSH, SW17 SW_PUSH, SW18 SW_PUSH, SW19 SW_PUSH, SW2 SW_PUSH, SW20 SW_PUSH, SW21 SW_PUSH, SW22 SW_PUSH, SW23 SW_PUSH, SW24 SW_PUSH, SW25 SW_PUSH, SW26 SW_PUSH, SW27 SW_PUSH, SW28 SW_PUSH, SW29 SW_PUSH, SW3 SW_PUSH, SW30 SW_PUSH, SW31 SW_PUSH, SW32 SW_PUSH, SW33 SW_PUSH, SW34 SW_PUSH, SW35 SW_PUSH, SW36 SW_PUSH, SW4 SW_PUSH, SW5 SW_PUSH, SW6 SW_PUSH, SW7 SW_PUSH, SW8 SW_PUSH, SW9 SW_PUSH, U1 ProMicro, U2 ProMicro

Commit message: changes
Parts:
- RSW2, RSW4: footprint kbd:Power -> Button_Switch_THT:SW_CuK_OS102011MA1QN1_SPDT_Angled
Changed lines of the file:
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@@
     (property "Reference" "RSW4" (id 0) (at 241.935 106.68 0))
     (property "Value" "SW_SPDT" (id 1) (at 241.935 109.22 0))
-    (property "Footprint" "kbd:Power" (id 2) (at 241.935 114.3 0)
+    (property "Footprint" "Button_Switch_THT:SW_CuK_OS102011MA1QN1_SPDT_Angled" (id 2) (at 241.935 114.3 0)
       (effects (font (size 1.27 1.27)) hide)
     )
@@
     (property "Reference" "RSW2" (id 0) (at 164.465 102.87 0))
     (property "Value" "SW_SPDT" (id 1) (at 164.465 105.41 0))
-    (property "Footprint" "kbd:Power" (id 2) (at 164.465 110.49 0)
+    (property "Footprint" "Button_Switch_THT:SW_CuK_OS102011MA1QN1_SPDT_Angled" (id 2) (at 164.465 110.49 0)
       (effects (font (size 1.27 1.27)) hide)
     )
@@
   (symbol (lib_id "power:GNDA") (at 247.015 114.3 0) (unit 1)
     (in_bom yes) (on_board yes)
-    (property "Reference" "#PWR?" (id 0) (at 247.015 120.65 0)
+    (property "Reference" "#PWR0119" (id 0) (at 247.015 120.65 0)
       (effects (font (size 1.27 1.27)) hide)
     )
@@
       (reference "#PWR0118") (unit 1) (value "VDD") (footprint "")
     )
+    (path "/f29568a0-1ec1-42ff-905c-80b34769e09a"
+      (reference "#PWR0119") (unit 1) (value "GNDA") (footprint "")
+    )
     (path "/1b14a23a-a1e4-4f61-b7c6-ed0f52a809c1"
       (reference "#PWR0120") (unit 1) (value "GNDA") (footprint "")
@@
       (reference "#PWR0122") (unit 1) (value "GNDA") (footprint "")
     )
-    (path "/f29568a0-1ec1-42ff-905c-80b34769e09a"
-      (reference "#PWR?") (unit 1) (value "GNDA") (footprint "")
-    )
     (path "/462d22f2-86b2-4b4c-9247-161cd747f1dd"
       (reference "BT1") (unit 1) (value "Battery_Cell") (footprint "kbd:Battery_pads")
@@
     )
     (path "/2b4cd6f8-610c-4bed-82fb-80f1c198ef79"
-      (reference "RSW2") (unit 1) (value "SW_SPDT") (footprint "kbd:Power")
+      (reference "RSW2") (unit 1) (value "SW_SPDT") (footprint "Button_Switch_THT:SW_CuK_OS102011MA1QN1_SPDT_Angled")
     )
     (path "/29ac1228-48da-4502-883d-75bf99318acd"
@@
     )
     (path "/108f5211-f2b2-456f-a4f6-42a19533a817"
-      (reference "RSW4") (unit 1) (value "SW_SPDT") (footprint "kbd:Power")
+      (reference "RSW4") (unit 1) (value "SW_SPDT") (footprint "Button_Switch_THT:SW_CuK_OS102011MA1QN1_SPDT_Angled")
     )
     (path "/da8e60a0-73b4-45a9-9589-4af5241172ba"
